Commit message: updated urdf

File: 3d_walker.urdf (robot description, URDF)
Before this commit: robot KneedCompassGait, 19 links, 16 joints
Joints:
- added joint left_hip_z_upperleg: type continuous, parent left_hip_z, child left_upper_leg, axis 0 0 1, limit effort=500
- added joint right_hip_z_upperleg: type continuous, parent right_hip_z, child right_upper_leg, axis 0 0 1, limit effort=500
- joint left_hip_x: child left_hip_y -> left_hip_x
- joint left_hip_y: child left_hip_z -> left_hip_y
- joint left_hip_z: child left_upper_leg -> left_hip_z
- joint right_hip_x: child right_hip_y -> right_hip_x
- joint right_hip_y: child right_hip_z -> right_hip_y
- joint right_hip_z: child right_upper_leg -> right_hip_z
